Commit message: adjusted the urdf so it looks nice in moveit setup assistant... not sure it's working though ;)

File: pa10_description/urdf/Mitsubishi-PA10_generated.urdf (robot description, URDF)
Before this commit: robot Mitsubishi-PA10, 8 links, 7 joints
Links:
- link link0: geometry collision mesh filename=file:///tmp/link0_mesh.dae scale=1 1 1; visual mesh filename=file:///tmp/link0_mesh.dae scale=1 1 1
- link link1: geometry collision mesh filename=file:///tmp/link1_mesh.dae scale=1 1 1; visual mesh filename=file:///tmp/link1_mesh.dae scale=1 1 1
- link link2: geometry collision mesh filename=file:///tmp/link2_mesh.dae scale=1 1 1; visual mesh filename=file:///tmp/link2_mesh.dae scale=1 1 1
- link link3: geometry collision mesh filename=file:///tmp/link3_mesh.dae scale=1 1 1; visual mesh filename=file:///tmp/link3_mesh.dae scale=1 1 1
- link link4: geometry collision mesh filename=file:///tmp/link4_mesh.dae scale=1 1 1; visual mesh filename=file:///tmp/link4_mesh.dae scale=1 1 1
- link link5: geometry collision mesh filename=file:///tmp/link5_mesh.dae scale=1 1 1; visual mesh filename=file:///tmp/link5_mesh.dae scale=1 1 1
- link link6: geometry collision mesh filename=file:///tmp/link6_mesh.dae scale=1 1 1; visual mesh filename=file:///tmp/link6_mesh.dae scale=1 1 1
- link link7: geometry collision mesh filename=file:///tmp/link7_mesh.dae scale=1 1 1; visual mesh filename=file:///tmp/link7_mesh.dae scale=1 1 1
Joints:
- joint E1: origin xyz=0 0 0.450 rpy=0 -0 0  -> xyz=0 0 0 rpy=0 -0 0 
- joint S1: origin xyz=0 0 0.315 rpy=0 -0 0  -> xyz=0 0 0 rpy=0 -0 0 
- joint W1: origin xyz=0 0 0.5 rpy=0 -0 0  -> xyz=0 0 0 rpy=0 -0 0 
