Commit message: Updated urdf for pa10

File: pa10_description/urdf/pa10.urdf (robot description, URDF)
Before this commit: robot pa10, 8 links, 7 joints
Links:
- link link0: mass None -> 1; geometry collision mesh filename=package://pa10_description/meshes/pa10/collision/link0_mesh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 scale=1 1 1; visual mesh filename=package://pa10_description/meshes/pa10/visual/link0_mesh.stl scale=1 1 1
- link link1: geometry collision mesh filename=package://pa10_description/meshes/pa10/collision/link1_mesh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 scale=1 1 1; visual mesh filename=package://pa10_description/meshes/pa10/visual/link1_mesh.stl scale=1 1 1
- link link2: geometry collision mesh filename=package://pa10_description/meshes/pa10/collision/link2_mesh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 scale=1 1 1; visual mesh filename=package://pa10_description/meshes/pa10/visual/link2_mesh.stl scale=1 1 1
- link link3: geometry collision mesh filename=package://pa10_description/meshes/pa10/collision/link3_mesh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 scale=1 1 1; visual mesh filename=package://pa10_description/meshes/pa10/visual/link3_mesh.stl scale=1 1 1
- link link4: geometry collision mesh filename=package://pa10_description/meshes/pa10/collision/link4_mesh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 scale=1 1 1; visual mesh filename=package://pa10_description/meshes/pa10/visual/link4_mesh.stl scale=1 1 1
- link link5: geometry collision mesh filename=package://pa10_description/meshes/pa10/collision/link5_mesh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 scale=1 1 1; visual mesh filename=package://pa10_description/meshes/pa10/visual/link5_mesh.stl scale=1 1 1
- link link6: geometry collision mesh filename=package://pa10_description/meshes/pa10/collision/link6_mesh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 scale=1 1 1; visual mesh filename=package://pa10_description/meshes/pa10/visual/link6_mesh.stl scale=1 1 1
- link link7: geometry collision mesh filename=package://pa10_description/meshes/pa10/collision/link7_mesh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 scale=1 1 1; visual mesh filename=package://pa10_description/meshes/pa10/collision/link7_mesh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 scale=1 1 1
Joints:
- removed joint joint_1
- removed joint joint_2
- removed joint joint_3
- removed joint joint_4
- removed joint joint_5
- removed joint joint_6
- removed joint joint_7
- added joint E1: type revolute, parent link3, child link4, origin xyz=0 0 0 rpy=0 -0 0 , axis 0 1 0, limit lower=-2.3911 upper=2.3911 effort=100000 velocity=0.5
- added joint E2: type revolute, parent link4, child link5, origin xyz=0 0 0 rpy=0 -0 0 , axis 0 0 1, limit lower=-4.45059 upper=4.45059 effort=100000 velocity=0.5
- added joint S1: type revolute, parent link0, child link1, origin xyz=0 0 0 rpy=0 -0 0 , axis 0 0 1, limit lower=-3.08923 upper=3.08923 effort=100000 velocity=0.5
- added joint S2: type revolute, parent link1, child link2, origin xyz=0 0 0 rpy=0 -0 0 , axis 0 1 0, limit lower=-1.58825 upper=1.58825 effort=100000 velocity=0.5
- added joint S3: type revolute, parent link2, child link3, origin xyz=0 0 0 rpy=0 -0 0 , axis 0 0 1, limit lower=-3.03687 upper=3.03687 effort=100000 velocity=0.5
- added joint W1: type revolute, parent link5, child link6, origin xyz=0 0 0 rpy=0 -0 0 , axis 0 1 0, limit lower=-2.87979 upper=2.87979 effort=100000 velocity=0.5
- added joint W2: type continuous, parent link6, child link7, origin xyz=0 0 1.35 rpy=0 -0 0 , axis 0 0 1, limit lower=-3.14159 upper=3.14159 effort=100000 velocity=0.5

Commit message: Revert "Updated urdf for pa10"
This reverts commit 83f6c0cf56bf1a2af740ef7bf310897c34f71236.

File: pa10_description/urdf/pa10.urdf (robot description, URDF)
Before this commit: robot Mitsubishi-PA10, 8 links, 7 joints
Links:
- link link0: mass 1 -> None; geometry collision mesh filename=package://pa10_description/meshes/pa10/collision/link0_mesh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 scale=1 1 1; visual mesh filename=package://pa10_description/meshes/pa10/visual/link0_mesh.dae scale=1 1 1
- link link1: geometry collision mesh filename=package://pa10_description/meshes/pa10/collision/link1_mesh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 scale=1 1 1; visual mesh filename=package://pa10_description/meshes/pa10/visual/link1_mesh.dae scale=1 1 1
- link link2: geometry collision mesh filename=package://pa10_description/meshes/pa10/collision/link2_mesh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 scale=1 1 1; visual mesh filename=package://pa10_description/meshes/pa10/visual/link2_mesh.dae scale=1 1 1
- link link3: geometry collision mesh filename=package://pa10_description/meshes/pa10/collision/link3_mesh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 scale=1 1 1; visual mesh filename=package://pa10_description/meshes/pa10/visual/link3_mesh.dae scale=1 1 1
- link link4: geometry collision mesh filename=package://pa10_description/meshes/pa10/collision/link4_mesh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 scale=1 1 1; visual mesh filename=package://pa10_description/meshes/pa10/visual/link4_mesh.dae scale=1 1 1
- link link5: geometry collision mesh filename=package://pa10_description/meshes/pa10/collision/link5_mesh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 scale=1 1 1; visual mesh filename=package://pa10_description/meshes/pa10/visual/link5_mesh.dae scale=1 1 1
- link link6: geometry collision mesh filename=package://pa10_description/meshes/pa10/collision/link6_mesh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 scale=1 1 1; visual mesh filename=package://pa10_description/meshes/pa10/visual/link6_mesh.dae scale=1 1 1
- link link7: geometry collision mesh filename=package://pa10_description/meshes/pa10/collision/link7_mesh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 scale=1 1 1; visual mesh filename=package://pa10_description/meshes/pa10/visual/link7_mesh.dae scale=1 1 1
Joints:
- removed joint E1
- removed joint E2
- removed joint S1
- removed joint S2
- removed joint S3
- removed joint W1
- removed joint W2
- added joint joint_1: type revolute, parent link0, child link1, origin xyz=0 0 0.315 rpy=0 -0 0 , axis 0 0 1, limit lower=-3.08923 upper=3.08923 effort=100000 velocity=0.4
- added joint joint_2: type revolute, parent link1, child link2, origin xyz=0 0 0 rpy=0 -0 0 , axis 0 1 0, limit lower=-1.58825 upper=1.58825 effort=100000 velocity=0.4
- added joint joint_3: type revolute, parent link2, child link3, origin xyz=0 0 0 rpy=0 -0 0 , axis 0 0 1, limit lower=-3.03687 upper=3.03687 effort=100000 velocity=0.5
- added joint joint_4: type revolute, parent link3, child link4, origin xyz=0 0 0.450 rpy=0 -0 0 , axis 0 1 0, limit lower=-2.3911 upper=2.3911 effort=100000 velocity=0.5
- added joint joint_5: type revolute, parent link4, child link5, origin xyz=0 0 0 rpy=0 -0 0 , axis 0 0 1, limit lower=-4.45059 upper=4.45059 effort=100000 velocity=0.5
- added joint joint_6: type revolute, parent link5, child link6, origin xyz=0 0 0.5 rpy=0 -0 0 , axis 0 1 0, limit lower=-2.87979 upper=2.87979 effort=100000 velocity=0.5
- added joint joint_7: type continuous, parent link6, child link7, origin xyz=0 0 0.085 rpy=0 -0 0 , axis 0 0 1, limit lower=-3.14159 upper=3.14159 effort=100000 velocity=0.5

Commit message: resette pa10.urdf to working version... changed to use stl in visual

File: pa10_description/urdf/pa10.urdf (robot description, URDF)
Before this commit: robot pa10, 8 links, 7 joints
Links:
- link link0: geometry collision mesh filename=package://pa10_description/meshes/pa10/collision/link0_mesh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 scale=1 1 1; visual mesh filename=package://pa10_description/meshes/pa10/visual/link0_mesh.stl scale=1 1 1
- link link1: geometry collision mesh filename=package://pa10_description/meshes/pa10/collision/link1_mesh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 scale=1 1 1; visual mesh filename=package://pa10_description/meshes/pa10/visual/link1_mesh.stl scale=1 1 1
- link link2: geometry collision mesh filename=package://pa10_description/meshes/pa10/collision/link2_mesh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 scale=1 1 1; visual mesh filename=package://pa10_description/meshes/pa10/visual/link2_mesh.stl scale=1 1 1
- link link3: geometry collision mesh filename=package://pa10_description/meshes/pa10/collision/link3_mesh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 scale=1 1 1; visual mesh filename=package://pa10_description/meshes/pa10/visual/link3_mesh.stl scale=1 1 1
- link link4: geometry collision mesh filename=package://pa10_description/meshes/pa10/collision/link4_mesh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 scale=1 1 1; visual mesh filename=package://pa10_description/meshes/pa10/visual/link4_mesh.stl scale=1 1 1
- link link5: geometry collision mesh filename=package://pa10_description/meshes/pa10/collision/link5_mesh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 scale=1 1 1; visual mesh filename=package://pa10_description/meshes/pa10/visual/link5_mesh.stl scale=1 1 1
- link link6: geometry collision mesh filename=package://pa10_description/meshes/pa10/collision/link6_mesh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 scale=1 1 1; visual mesh filename=package://pa10_description/meshes/pa10/visual/link6_mesh.stl scale=1 1 1
- link link7: geometry collision mesh filename=package://pa10_description/meshes/pa10/collision/link7_mesh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 scale=1 1 1; visual mesh filename=package://pa10_description/meshes/pa10/visual/link7_mesh.stl scale=1 1 1
