Commit message: xacro for pa10_description, model loads now in gazebo, world file needs to be adapted

File: pa10_description/urdf/pa10.xacro (robot description, xacro)
@@ -1,4 +1,14 @@
 <?xml version="1.0"?>
-<robot name="pa10">
+<robot name="pa10" xmlns:xacro="http://www.ros.org/wiki/xacro">
+  <!-- Import all Gazebo-customization elements, including Gazebo colors -->
+  <xacro:include filename="$(find pa10_description)/urdf/pa10.gazebo" />
+  <!-- Import Rviz colors -->
+  <xacro:include filename="$(find pa10_description)/urdf/materials.xacro" />
+  <!-- Used for fixing robot to Gazebo 'base_link' -->
+  <link name="world"/>
+  <joint name="fixed" type="fixed">
+    <parent link="world"/>
+    <child link="link0"/>
+  </joint>
   <link name="link0">
     <visual>
@@ -7,7 +17,5 @@
         <mesh filename="package://pa10_description/meshes/pa10/visual/link0_mesh.stl" scale="1 1 1" />
       </geometry>
-      <material name="cyan">
-        <color rgba="0.35 0.5 0.35 1"/>
-      </material>
+      <material name="cyan" />
     </visual>
     <collision>
@@ -17,4 +25,9 @@
       </geometry>
     </collision>
+    <inertial>
+      <mass value="1" />
+      <origin xyz="0 0 0" rpy="0 -0 0"/>
+      <inertia ixx="1" ixy="0" ixz="0" iyy="1" iyz="0" izz="1"/>
+    </inertial>
   </link>
   <link name="link1">
@@ -24,7 +37,5 @@
         <mesh filename="package://pa10_description/meshes/pa10/visual/link1_mesh.stl" scale="1 1 1" />
       </geometry>
-      <material name="grey">
-        <color rgba=".6 .6 .6 1"/>
-      </material>
+      <material name="grey" />
     </visual>
     <collision>

Commit message: pa10_description + moveit_config with pg70 gripper

File: pa10_description/urdf/pa10.xacro (robot description, xacro)
@@ -5,4 +5,6 @@
   <!-- Import Rviz colors -->
   <xacro:include filename="$(find pa10_description)/urdf/materials.xacro" />
+  <!-- Import gripper -->
+  <xacro:include filename="$(find schunk_description)/urdf/pg70/pg70.urdf.xacro" />
   <!-- Used for fixing robot to Gazebo 'base_link' -->
   <link name="world"/>
@@ -227,3 +229,7 @@
     <dynamics damping="0.2" friction="0" />
   </joint>
+  <!-- gripper -->
+  <xacro:schunk_pg70 name="gripper" parent="link7">
+      <origin xyz="0 0 0.02" rpy="0 0 0" />
+  </xacro:schunk_pg70>
 </robot>

Commit message: increased robot z-position, moveit_config changes

File: pa10_description/urdf/pa10.xacro (robot description, xacro)
@@ -12,4 +12,5 @@
     <parent link="world"/>
     <child link="link0"/>
+    <origin rpy="0 0 0.523" xyz="0 0 .3"/>
   </joint>
   <link name="link0">
@@ -228,4 +229,5 @@
     <limit lower="-3.14159" upper="3.14159" effort="100000" velocity="0.5" />
     <dynamics damping="0.2" friction="0" />
+    <!--<safety_controller k_position="100" k_velocity="1.5" soft_lower_limit="-2.857" soft_upper_limit="2.857"/>-->
   </joint>
   <!-- gripper -->

Commit message: Scene update

File: pa10_description/urdf/pa10.xacro (robot description, xacro)
@@ -12,5 +12,5 @@
     <parent link="world"/>
     <child link="link0"/>
-    <origin rpy="0 0 0.523" xyz="0 0 .3"/>
+    <origin rpy="0 0 0.523" xyz="0 0 .79"/>
   </joint>
   <link name="link0">
